File: Schematic_PCB/Music_Visualizer/Music_Visualizer.kicad_sch (KiCad schematic)
At the start: 48 parts, among them J1 AudioJack3, J3 Screw_Terminal_01x02, SW1 SW_SPDT, U1 LM324, U2 LM324, U3 LM324, U4 LM324, U5 LM324, U6 LM324, U7 LM324

Commit message: Change freq ranges to quasi-log
Other:
- note added: "Bass: [60Hz:150Hz]"
- note added: "Low Midrange: [150Hz:400Hz]"
- note added: "Midrange: [400Hz:1kHz]"
- note added: "Presence: [2.5kHz:6kHz]"
- note added: "Upper-Midrange: [1kHz:2.5kHz]"
- note removed: "Bass: [60Hz:250Hz]"
- note removed: "Low Midrange: [250Hz:500Hz]"
- note removed: "Midrange: [500Hz:2kHz]"
- note removed: "Presence: [4kHz:6kHz]"
- note removed: "Upper-Midrange: [2kHz:4kHz]"
- moved on the sheet: C1, C2, C3, C4, C43, C5, C6, R1, R2, R3, R4, R5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

Commit message: Add output buffer
Parts:
- removed J1: AudioJack3, Connector_Audio:Jack_3.5mm_CUI_SJ-3523-SMT_Horizontal, symbol Connector:AudioJack3
- removed SW1: SW_SPDT, Slide_Switch:SW_OS102011MS2QN1, symbol Switch:SW_SPDT
- added C7: 100n, Capacitor_SMD:C_0603_1608Metric_Pad1.08x0.95mm_HandSolder, symbol Device:C
- added C8: 1u, Capacitor_SMD:C_0603_1608Metric_Pad1.08x0.95mm_HandSolder, symbol Device:C
- added J1, J4: NMJ4HCD2, Connector_Audio:Jack_6.35mm_Neutrik_NMJ4HCD2_Horizontal, symbol Connector_Audio:NMJ4HCD2
- added J5: Screw_Terminal_01x02, TerminalBlock_Phoenix:TerminalBlock_Phoenix_MPT-0,5-2-2.54_1x02_P2.54mm_Horizontal, symbol Connector:Screw_Terminal_01x02
- added R11: 1m, Resistor_SMD:R_0603_1608Metric_Pad0.98x0.95mm_HandSolder, symbol Device:R
- added R12: 10k, Resistor_SMD:R_0603_1608Metric_Pad0.98x0.95mm_HandSolder, symbol Device:R
- added unit 4 of U3
Connections:
- net Vsig_male is gone; now on net GND: J3.2 (Pin_2)
- net GND: now also J1.S, J1.SN, J4.S, J4.SN, J5.2 (Pin_2), R12.2; no longer J3.1 (Pin_1)
- net VCC4_5: now also R11.2
- net at C9.1: now also J4.T
- new net: C7.2, R11.1, U3.12 (+)
- new net: C8.1, U3.13 (-), U3.14
- new net: J1.TN, J5.1 (Pin_1)
- new net: C8.2, J1.T, R12.1
- new net: J3.1 (Pin_1), J4.TN
Other:
- note added: "Todo: -add dc decoupling for all inputs and dividers 1uf - replace all filters with standertised capacitors ( maybe capacitor arrays) - replace footprints Done --replace -5v with voltage divider and unity gain amp-"
- note removed: "Todo: -add dc decoupling for all inputs and dividers 1uf - replace all filters with standertised capacitors ( maybe capacitor arrays) Done --replace -5v with voltage divider and unity gain amp-"
- moved on the sheet: C10, C9, J3, R10, U2D

Commit message: Add filters with new values
Parts:
- added C11, C12, C13, C14: 100n, Capacitor_SMD:C_0603_1608Metric_Pad1.08x0.95mm_HandSolder, symbol Device:C
- added C15, C16: 100n, Capacitor_SMD:C_1206_3216Metric, symbol Device:C
- added C17, C24, C31, C38, C46, C53: 100u, Capacitor_SMD:C_1206_3216Metric, symbol Device:C
- added C18, C19, C20, C21: 47n, Capacitor_SMD:C_0603_1608Metric_Pad1.08x0.95mm_HandSolder, symbol Device:C
- added C22, C23: 47n, Capacitor_SMD:C_1206_3216Metric, symbol Device:C
- added C25, C26, C27, C28: 22n, Capacitor_SMD:C_0603_1608Metric_Pad1.08x0.95mm_HandSolder, symbol Device:C
- added C29, C30: 22n, Capacitor_SMD:C_1206_3216Metric, symbol Device:C
- added C32, C33, C34, C35: 10n, Capacitor_SMD:C_0603_1608Metric_Pad1.08x0.95mm_HandSolder, symbol Device:C
- added C36, C37: 10n, Capacitor_SMD:C_1206_3216Metric, symbol Device:C
- added C39, C40, C41, C42: 4.7n, Capacitor_SMD:C_0603_1608Metric_Pad1.08x0.95mm_HandSolder, symbol Device:C
- added C44, C45: 4.7n, Capacitor_SMD:C_1206_3216Metric, symbol Device:C
- added C47, C48, C49, C50: 2.2n, Capacitor_SMD:C_0603_1608Metric_Pad1.08x0.95mm_HandSolder, symbol Device:C
- added C51, C52: 2.2n, Capacitor_SMD:C_1206_3216Metric, symbol Device:C
- added R13: 26.6k, Resistor_SMD:R_0603_1608Metric_Pad0.98x0.95mm_HandSolder, symbol Device:R
- added R14, R46: 7k, Resistor_SMD:R_0603_1608Metric_Pad0.98x0.95mm_HandSolder, symbol Device:R
- added R15: 115k, Resistor_SMD:R_0603_1608Metric_Pad0.98x0.95mm_HandSolder, symbol Device:R
- added R16: 11.7k, Resistor_SMD:R_0603_1608Metric_Pad0.98x0.95mm_HandSolder, symbol Device:R
- added R17, R67: 3k, Resistor_SMD:R_0603_1608Metric_Pad0.98x0.95mm_HandSolder, symbol Device:R
- added R18: 51k, Resistor_SMD:R_0603_1608Metric_Pad0.98x0.95mm_HandSolder, symbol Device:R
- added R19: 17.7k, Resistor_SMD:R_0603_1608Metric_Pad0.98x0.95mm_HandSolder, symbol Device:R
- added R20: 14.5k, Resistor_SMD:R_0603_1608Metric_Pad0.98x0.95mm_HandSolder, symbol Device:R
- added R21: 35.4k, Resistor_SMD:R_0603_1608Metric_Pad0.98x0.95mm_HandSolder, symbol Device:R
- added R22, R32, R42, R52, R62, R73: 1k, Resistor_SMD:R_0603_1608Metric_Pad0.98x0.95mm_HandSolder, symbol Device:R
- added R23: 21k, Resistor_SMD:R_0603_1608Metric_Pad0.98x0.95mm_HandSolder, symbol Device:R
- added R24, R56: 6.5k, Resistor_SMD:R_0603_1608Metric_Pad0.98x0.95mm_HandSolder, symbol Device:R
- added R25: 92.4k, Resistor_SMD:R_0603_1608Metric_Pad0.98x0.95mm_HandSolder, symbol Device:R
- added R26, R50: 8.7k, Resistor_SMD:R_0603_1608Metric_Pad0.98x0.95mm_HandSolder, symbol Device:R
- added R27: 2.7k, Resistor_SMD:R_0603_1608Metric_Pad0.98x0.95mm_HandSolder, symbol Device:R
- added R28: 38.3k, Resistor_SMD:R_0603_1608Metric_Pad0.98x0.95mm_HandSolder, symbol Device:R
- added R29: 13.5k, Resistor_SMD:R_0603_1608Metric_Pad0.98x0.95mm_HandSolder, symbol Device:R
- added R30: 14.7k, Resistor_SMD:R_0603_1608Metric_Pad0.98x0.95mm_HandSolder, symbol Device:R
- added R31: 27.1k, Resistor_SMD:R_0603_1608Metric_Pad0.98x0.95mm_HandSolder, symbol Device:R
- added R33: 18.2k, Resistor_SMD:R_0603_1608Metric_Pad0.98x0.95mm_HandSolder, symbol Device:R
- added R34: 4.7k, Resistor_SMD:R_0603_1608Metric_Pad0.98x0.95mm_HandSolder, symbol Device:R
- added R35: 78k, Resistor_SMD:R_0603_1608Metric_Pad0.98x0.95mm_HandSolder, symbol Device:R
- added R36: 8k, Resistor_SMD:R_0603_1608Metric_Pad0.98x0.95mm_HandSolder, symbol Device:R
- added R37: 2.1k, Resistor_SMD:R_0603_1608Metric_Pad0.98x0.95mm_HandSolder, symbol Device:R
- added R38: 34.7k, Resistor_SMD:R_0603_1608Metric_Pad0.98x0.95mm_HandSolder, symbol Device:R
- added R39: 12.1k, Resistor_SMD:R_0603_1608Metric_Pad0.98x0.95mm_HandSolder, symbol Device:R
- added R40: 9.9k, Resistor_SMD:R_0603_1608Metric_Pad0.98x0.95mm_HandSolder, symbol Device:R
- added R41: 24.1k, Resistor_SMD:R_0603_1608Metric_Pad0.98x0.95mm_HandSolder, symbol Device:R
- added R43: 16k, Resistor_SMD:R_0603_1608Metric_Pad0.98x0.95mm_HandSolder, symbol Device:R
- added R44: 4.2k, Resistor_SMD:R_0603_1608Metric_Pad0.98x0.95mm_HandSolder, symbol Device:R
- added R45: 69.3k, Resistor_SMD:R_0603_1608Metric_Pad0.98x0.95mm_HandSolder, symbol Device:R
- added R47: 1.8k, Resistor_SMD:R_0603_1608Metric_Pad0.98x0.95mm_HandSolder, symbol Device:R
- added R48: 30.6k, Resistor_SMD:R_0603_1608Metric_Pad0.98x0.95mm_HandSolder, symbol Device:R
- added R49: 10.6k, Resistor_SMD:R_0603_1608Metric_Pad0.98x0.95mm_HandSolder, symbol Device:R
- added R51: 21.2k, Resistor_SMD:R_0603_1608Metric_Pad0.98x0.95mm_HandSolder, symbol Device:R
- added R53: 14.3k, Resistor_SMD:R_0603_1608Metric_Pad0.98x0.95mm_HandSolder, symbol Device:R
- added R54: 3.3k, Resistor_SMD:R_0603_1608Metric_Pad0.98x0.95mm_HandSolder, symbol Device:R
- added R55: 61.6k, Resistor_SMD:R_0603_1608Metric_Pad0.98x0.95mm_HandSolder, symbol Device:R
- added R57: 1.5k, Resistor_SMD:R_0603_1608Metric_Pad0.98x0.95mm_HandSolder, symbol Device:R
- added R58: 28.2k, Resistor_SMD:R_0603_1608Metric_Pad0.98x0.95mm_HandSolder, symbol Device:R
- added R59: 9.7k, Resistor_SMD:R_0603_1608Metric_Pad0.98x0.95mm_HandSolder, symbol Device:R
- added R60: 6.7k, Resistor_SMD:R_0603_1608Metric_Pad0.98x0.95mm_HandSolder, symbol Device:R
- added R61: 19.4k, Resistor_SMD:R_0603_1608Metric_Pad0.98x0.95mm_HandSolder, symbol Device:R
- added R63: 8.9k, Resistor_SMD:R_0603_1608Metric_Pad0.98x0.95mm_HandSolder, symbol Device:R
- added R64: 4.9k, Resistor_SMD:R_0603_1608Metric_Pad0.98x0.95mm_HandSolder, symbol Device:R
- added R65: 41.3k, Resistor_SMD:R_0603_1608Metric_Pad0.98x0.95mm_HandSolder, symbol Device:R
- added R68: 1.6k, Resistor_SMD:R_0603_1608Metric_Pad0.98x0.95mm_HandSolder, symbol Device:R
- added R69: 13.8k, Resistor_SMD:R_0603_1608Metric_Pad0.98x0.95mm_HandSolder, symbol Device:R
- added R70: 5.2k, Resistor_SMD:R_0603_1608Metric_Pad0.98x0.95mm_HandSolder, symbol Device:R
- added R71: 23k, Resistor_SMD:R_0603_1608Metric_Pad0.98x0.95mm_HandSolder, symbol Device:R
- added R72: 10.3k, Resistor_SMD:R_0603_1608Metric_Pad0.98x0.95mm_HandSolder, symbol Device:R
- added unit 4 of U4
- added unit 3 of U4
- added unit 2 of U4
- added unit 1 of U4
- added unit 3 of U5
- added unit 1 of U5
- added unit 4 of U5
- added unit 2 of U5
- added unit 4 of U6
- added unit 3 of U6
- added unit 2 of U6
- added unit 1 of U6
- added unit 3 of U7
- added unit 4 of U7
- added unit 2 of U7
- added unit 1 of U7
- added U8, U9: LM324, Package_SO:SOIC-14_3.9x8.7mm_P1.27mm, symbol Amplifier_Operational:LM324
Connections:
- net GND: now also R22.2, R32.2, R42.2, R52.2, R62.2, R73.2
- net VBass: now also C17.2, R22.1
- net VBrilliance: now also C53.2, R73.1
- net VCC4_5: now also R14.2, R17.2, R20.2, R24.2, R27.2, R30.2, R34.2, R37.2, R40.2, R44.2, R47.2, R50.2, R54.2, R57.2, R60.2, R64.2, R68.2, R71.2, U4.10 (+), U4.3 (+), U4.5 (+), U5.10 (+), U5.3 (+), U5.5 (+), U6.10 (+), U6.3 (+), U6.5 (+), U7.10 (+), U7.3 (+), U7.5 (+), U8.10 (+), U8.3 (+), U8.5 (+), U9.10 (+), U9.3 (+), U9.5 (+)
- net VLowerMidrange: now also C24.2, R32.1
- net VMidrange: now also C31.2, R42.1
- net VPresence: now also C46.2, R62.1
- net VUpperMidrange: now also C38.2, R52.1
- net Vsig: now also U4.12 (+), U5.12 (+), U6.12 (+), U7.12 (+), U8.12 (+), U9.12 (+)
- new net: R13.1, U4.13 (-), U4.14
- new net: C41.1, C42.1, R56.2, R57.1
- new net: C42.2, R58.2, U8.6 (-)
- new net: R33.1, U6.13 (-), U6.14
- new net: C25.1, C26.1, R33.2, R34.1
- new net: C26.2, R35.2, U6.2 (-)
- new net: C18.1, C19.1, R23.2, R24.1
- new net: C15.1, C16.1, R19.2, R20.1
- new net: C16.2, R21.2, U4.9 (-)
- new net: C22.2, C24.1, R31.1, U5.8
- new net: R43.1, U7.13 (-), U7.14
- new net: C32.1, C33.1, R43.2, R44.1
- new net: C51.1, C52.1, R70.2, R71.1
- new net: C52.2, R72.2, U9.9 (-)
- new net: C41.2, R58.1, R59.1, U8.7
- new net: C44.1, C45.1, R59.2, R60.1
- new net: C18.2, R25.1, R26.1, U5.1
- new net: C20.1, C21.1, R26.2, R27.1
- new net: C47.1, C48.1, R63.2, R64.1
- new net: C48.2, R65.2, U9.2 (-)
- new net: C25.2, R35.1, R36.1, U6.1
- new net: C19.2, R25.2, U5.2 (-)
- new net: R23.1, U5.13 (-), U5.14
- new net: C36.2, C38.1, R51.1, U7.8
- new net: C37.2, R51.2, U7.9 (-)
- new net: C23.2, R31.2, U5.9 (-)
- new net: C27.1, C28.1, R36.2, R37.1
- new net: C39.1, C40.1, R53.2, R54.1
- new net: C22.1, C23.1, R29.2, R30.1
- new net: C29.2, C31.1, R41.1, U6.8
- new net: C30.2, R41.2, U6.9 (-)
- new net: C49.1, C50.1, R67.2, R68.1
- new net: C49.2, R69.1, R70.1, U9.7
- new net: C11.1, C12.1, R13.2, R14.1
- new net: C12.2, R15.2, U4.2 (-)
- new net: C15.2, C17.1, R21.1, U4.8
- new net: C51.2, C53.1, R72.1, U9.8
- new net: C35.2, R48.2, U7.6 (-)
- new net: C34.2, R48.1, R49.1, U7.7
- new net: C32.2, R45.1, R46.1, U7.1
- new net: R63.1, U9.13 (-), U9.14
- new net: C40.2, R55.2, U8.2 (-)
- new net: C39.2, R55.1, R56.1, U8.1
- new net: C11.2, R15.1, R16.1, U4.1
- new net: C28.2, R38.2, U6.6 (-)
- new net: C44.2, C46.1, R61.1, U8.8
- new net: C45.2, R61.2, U8.9 (-)
- new net: C14.2, R18.2, U4.6 (-)
- new net: C13.2, R18.1, R19.1, U4.7
- new net: C27.2, R38.1, R39.1, U6.7
- new net: C13.1, C14.1, R16.2, R17.1
- new net: C34.1, C35.1, R46.2, R47.1
- new net: C29.1, C30.1, R39.2, R40.1
- new net: C20.2, R28.1, R29.1, U5.7
- new net: C47.2, R65.1, R67.1, U9.1
- new net: C21.2, R28.2, U5.6 (-)
- new net: C36.1, C37.1, R49.2, R50.1
- new net: C50.2, R69.2, U9.6 (-)
- new net: C33.2, R45.2, U7.2 (-)
- new net: R53.1, U8.13 (-), U8.14
Other:
- note removed: "Jamaina"

Commit message: Change op amp exit cap
Parts:
- removed C10, C8: 1u, Capacitor_SMD:C_0603_1608Metric_Pad1.08x0.95mm_HandSolder, symbol Device:C
- removed C60, C61, C62, C63, C64, C65, C66, C67, C68, C69, C70, C71, C72, C73: 0.1uF, Capacitor_SMD:C_0805_2012Metric, symbol Device:C
- removed C7, C9: 100n, Capacitor_SMD:C_0603_1608Metric_Pad1.08x0.95mm_HandSolder, symbol Device:C
- removed J1, J4: NMJ4HCD2, Connector_Audio:Jack_6.35mm_Neutrik_NMJ4HCD2_Horizontal, symbol Connector_Audio:NMJ4HCD2
- removed J3, J5: Screw_Terminal_01x02, TerminalBlock_Phoenix:TerminalBlock_Phoenix_MPT-0,5-2-2.54_1x02_P2.54mm_Horizontal, symbol Connector:Screw_Terminal_01x02
- removed R10, R11: 1m, Resistor_SMD:R_0603_1608Metric_Pad0.98x0.95mm_HandSolder, symbol Device:R
- removed R12: 10k, Resistor_SMD:R_0603_1608Metric_Pad0.98x0.95mm_HandSolder, symbol Device:R
- removed unit 5 of U1
- removed U2, U3: LM324, Package_SO:SOIC-14_3.9x8.7mm_P1.27mm, symbol Amplifier_Operational:LM324
- removed unit 5 of U4
- removed unit 5 of U5
- removed unit 5 of U6
- removed unit 5 of U7
- C1, C11, C12, C13, C14, C18, C19, C2, C20, C21, C25, C26, C27, C28, C3, C32, C33, C34, C35, C39, C4, C40, C41, C42, C47, C48, C49, C50: footprint Capacitor_SMD:C_0603_1608Metric_Pad1.08x0.95mm_HandSolder -> Capacitor_SMD:C_0805_2012Metric_Pad1.18x1.45mm_HandSolder
- C15, C16, C22, C23, C29, C30, C36, C37, C44, C45, C5, C51, C52, C6: footprint Capacitor_SMD:C_1206_3216Metric -> Capacitor_SMD:C_0805_2012Metric_Pad1.18x1.45mm_HandSolder
- C17, C24, C43: value 100u -> 10u; footprint Capacitor_SMD:C_1206_3216Metric -> Capacitor_SMD:C_0805_2012Metric_Pad1.18x1.45mm_HandSolder
- C31, C38, C46, C53: value 100u -> 1u; footprint Capacitor_SMD:C_1206_3216Metric -> Capacitor_SMD:C_0805_2012Metric_Pad1.18x1.45mm_HandSolder
- R1, R13, R14, R15, R16, R17, R18, R19, R2, R20, R21, R22, R23, R24, R25, R26, R27, R28, R29, R3, R30, R31, R32, R33, R34, R35, R36, R37, R38, R39, R4, R40, R41, R42, R43, R44, R45, R46, R47, R48, R49, R5, R50, R51, R52, R53, R54, R55, R56, R57, R58, R59, R6, R60, R61, R62, R63, R64, R65, R66, R67, R68, R69, R7, R70, R71, R72, R73, R8, R9: footprint Resistor_SMD:R_0603_1608Metric_Pad0.98x0.95mm_HandSolder -> Resistor_SMD:R_0805_2012Metric_Pad1.20x1.40mm_HandSolder
Other:
- added sheet Audio signal (audio_signal.kicad_sch)
- note added: "Todo: Done - replace all filters with standertised capacitors ( maybe capacitor arrays) - replace footprints --replace -5v with voltage divider and unity gain amp-"
- note removed: "Audio Signal Input"
- note removed: "De coupling, maybe 10uf Electro"
- note removed: "Input Buffer"
- note removed: "Op-Amp Power"
- note removed: "Todo: -add dc decoupling for all inputs and dividers 1uf - replace all filters with standertised capacitors ( maybe capacitor arrays) - replace footprints Done --replace -5v with voltage divider and unity gain amp-"

Commit message: Replace ideal resistors with aprox
Parts:
- R1: value 29.7k -> 27k
- R13: value 26.6k -> 27k
- R14, R46: value 7k -> 6.8k
- R15: value 115k -> 120k
- R16: value 11.7k -> 12k
- R17, R67: value 3k -> 3.3k
- R18: value 51k -> 56k
- R19: value 17.7k -> 18k
- R2: value 12.5k -> 12k
- R20: value 14.5k -> 15k
- R21: value 35.4k -> 39k
- R23: value 21k -> 22k
- R24, R56: value 6.5k -> 6.8k
- R25: value 92.4k -> 100k
- R26, R50: value 8.7k -> 8.2
- R28: value 38.3k -> 39k
- R29: value 13.5k -> 15k
- R3: value 133.9k -> 150k
- R30: value 14.7k -> 15k
- R31: value 27.1k -> 27k
- R33: value 18.2k -> 18k
- R35: value 78k -> 82k
- R36: value 8k -> 8.2k
- R37: value 2.1k -> 2.2k
- R38: value 34.7k -> 33k
- R39: value 12.1k -> 12k
- R4: value 11k -> 10k
- R40: value 9.9k -> 10k
- R41: value 24.1k -> 27k
- R43: value 16k -> 15k
- R44: value 4.2k -> 4.7k
- R45: value 69.3k -> 68k
- R48: value 30.6k -> 33k
- R49: value 10.6k -> 10k
- R5: value 4.6k -> 4.7k
- R51: value 21.2k -> 22k
- R53: value 14.3k -> 15k
- R55: value 61.6k -> 56k
- R58: value 28.2k -> 27k
- R59: value 9.7k -> 10k
- R6: value 49.5k -> 47k
- R60: value 6.7k -> 6.8k
- R61: value 19.4k -> 22k
- R63: value 8.9k -> 10k
- R64: value 4.9k -> 5.6k
- R65: value 41.3k -> 39k
- R69: value 13.8k -> 15k
- R70: value 5.2k -> 5.6k
- R71: value 23k -> 22k
- R72: value 10.3k -> 10k
- R8: value 36.4k -> 39k
- R9: value 36.2k -> 39k
Changed lines of the file:
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@@
 			)
 		)
-		(property "Value" "12.5k"
+		(property "Value" "12k"
 			(at 74.93 64.7699 0)
 			(effects
@@
 			)
 		)
-		(property "Value" "6.5k"
+		(property "Value" "6.8k"
 			(at 63.5 201.9299 0)
 			(effects
@@
 			)
 		)
-		(property "Value" "16k"
+		(property "Value" "15k"
 			(at 317.5 49.53 90)
 			(effects
@@
 			)
 		)
-		(property "Value" "9.7k"
+		(property "Value" "10k"
 			(at 420.37 127 90)
 			(effects
@@
 			)
 		)
-		(property "Value" "8.7k"
+		(property "Value" "8.2"
 			(at 110.49 195.58 90)
 			(effects
@@
 			)
 		)
-		(property "Value" "78k"
+		(property "Value" "82k"
 			(at 83.82 265.4299 0)
 			(effects
@@
 			)
 		)
-		(property "Value" "92.4k"
+		(property "Value" "100k"
 			(at 81.28 191.7699 0)
 			(effects
@@
 			)
 		)
-		(property "Value" "21k"
+		(property "Value" "22k"
 			(at 54.61 193.04 90)
 			(effects
@@
 			)
 		)
-		(property "Value" "133.9k"
+		(property "Value" "150k"
 			(at 92.71 54.6099 0)
 			(effects
@@
 			)
 		)
-		(property "Value" "2.1k"
+		(property "Value" "2.2k"
 			(at 123.19 278.1299 0)
 			(effects
@@
 			)
 		)
-		(property "Value" "4.2k"
+		(property "Value" "4.7k"
 			(at 326.39 58.4199 0)
 			(effects
@@
 			)
 		)
-		(property "Value" "6.5k"
+		(property "Value" "6.8k"
 			(at 372.11 127 90)
 			(effects
@@
 			)
 		)
-		(property "Value" "61.6k"
+		(property "Value" "56k"
 			(at 342.9 123.1899 0)
 			(effects
@@
 			)
 		)
-		(property "Value" "26.6k"
+		(property "Value" "27k"
 			(at 54.61 123.19 90)
 			(effects
@@
 			)
 		)
-		(property "Value" "115k"
+		(property "Value" "120k"
 			(at 81.28 121.9199 0)
 			(effects
@@
 			)
 		)
-		(property "Value" "14.5k"
+		(property "Value" "15k"
 			(at 168.91 134.6199 0)
 			(effects
@@
 			)
 		)
-		(property "Value" "6.7k"
+		(property "Value" "6.8k"
 			(at 430.53 135.8899 0)
 			(effects
@@
 			)
 		)
-		(property "Value" "23k"
+		(property "Value" "22k"
 			(at 430.53 209.5499 0)
 			(effects
@@
 			)
 		)
-		(property "Value" "3k"
+		(property "Value" "3.3k"
 			(at 120.65 134.6199 0)
 			(effects
@@
 			)
 		)
-		(property "Value" "7k"
+		(property "Value" "6.8k"
 			(at 373.38 52.07 90)
 			(effects
@@
 			)
 		)
-		(property "Value" "34.7k"
+		(property "Value" "33k"
 			(at 135.89 265.4299 0)
 			(effects
@@
 			)
 		)
-		(property "Value" "11k"
+		(property "Value" "10k"
 			(at 121.92 58.42 90)
 			(effects
@@
 			)
 		)
-		(property "Value" "19.4k"
+		(property "Value" "22k"
 			(at 445.77 123.1899 0)
 			(effects
@@
 			)
 		)
-		(property "Value" "11.7k"
+		(property "Value" "12k"
 			(at 110.49 125.73 90)
 			(effects
@@
 			)
 		)
-		(property "Value" "24.1k"
+		(property "Value" "27k"
 			(at 186.69 265.4299 0)
 			(effects
@@
 			)
 		)
-		(property "Value" "28.2k"
+		(property "Value" "27k"
 			(at 394.97 123.1899 0)
 			(effects
@@
 			)
 		)
-		(property "Value" "3k"
+		(property "Value" "3.3k"
 			(at 372.11 200.66 90)
 			(effects
@@
 			)
 		)
-		(property "Value" "4.9k"
+		(property "Value" "5.6k"
 			(at 325.12 207.0099 0)
 			(effects
@@
 			)
 		)
-		(property "Value" "4.6k"
+		(property "Value" "4.7k"
 			(at 132.08 67.3099 0)
 			(effects
@@
 			)
 		)
-		(property "Value" "30.6k"
+		(property "Value" "33k"
 			(at 396.24 48.2599 0)
 			(effects
@@
 			)
 		)
-		(property "Value" "8.7k"
+		(property "Value" "8.2"
 			(at 431.8 60.9599 0)
 			(effects
@@
 			)
 		)
-		(property "Value" "13.8k"
+		(property "Value" "15k"
 			(at 394.97 196.8499 0)
 			(effects
@@
 			)
 		)
-		(property "Value" "38.3k"
+		(property "Value" "39k"
 			(at 133.35 191.7699 0)
 			(effects
@@
 			)
 		)
-		(property "Value" "18.2k"
+		(property "Value" "18k"
 			(at 57.15 266.7 90)
 			(effects
@@
 			)
 		)
-		(property "Value" "9.9k"
+		(property "Value" "10k"
 			(at 171.45 278.1299 0)
 			(effects
@@
 			)
 		)
-		(property "Value" "69.3k"
+		(property "Value" "68k"
 			(at 344.17 48.2599 0)
 			(effects
@@
 			)
 		)
-		(property "Value" "5.2k"
+		(property "Value" "5.6k"
 			(at 420.37 200.66 90)
 			(effects
@@
 			)
 		)
-		(property "Value" "12.1k"
+		(property "Value" "12k"
 			(at 161.29 269.24 90)
 			(effects
@@
 			)
 		)
-		(property "Value" "10.6k"
+		(property "Value" "10k"
 			(at 421.64 52.07 90)
 			(effects
@@
 			)
 		)
-		(property "Value" "35.4k"
+		(property "Value" "39k"
 			(at 184.15 121.9199 0)
 			(effects
@@
 			)
 		)
-		(property "Value" "7k"
+		(property "Value" "6.8k"
 			(at 63.5 132.0799 0)
 			(effects
@@
 			)
 		)
-		(property "Value" "41.3k"
+		(property "Value" "39k"
 			(at 342.9 196.8499 0)
 			(effects
@@
 			)
 		)
-		(property "Value" "17.7k"
+		(property "Value" "18k"
 			(at 158.75 125.73 90)
 			(effects
@@
 			)
 		)
-		(property "Value" "8.9k"
+		(property "Value" "10k"
 			(at 316.23 198.12 90)
 			(effects
@@
 			)
 		)
-		(property "Value" "13.5k"
+		(property "Value" "15k"
 			(at 158.75 195.58 90)
 			(effects
@@
 			)
 		)
-		(property "Value" "29.7k"
+		(property "Value" "27k"
 			(at 66.04 55.88 90)
 			(effects
@@
 			)
 		)
-		(property "Value" "21.2k"
+		(property "Value" "22k"
 			(at 447.04 48.2599 0)
 			(effects
@@
 			)
 		)
-		(property "Value" "14.3k"
+		(property "Value" "15k"
 			(at 316.23 124.46 90)
 			(effects
@@
 			)
 		)
-		(property "Value" "36.4k"
+		(property "Value" "39k"
 			(at 180.34 67.3099 0)
 			(effects
@@
 			)
 		)
-		(property "Value" "8k"
+		(property "Value" "8.2k"
 			(at 113.03 269.24 90)
 			(effects
@@
 			)
 		)
-		(property "Value" "10.3k"
+		(property "Value" "10k"
 			(at 445.77 196.8499 0)
 			(effects
@@
 			)
 		)
-		(property "Value" "49.5k"
+		(property "Value" "47k"
 			(at 144.78 54.6099 0)
 			(effects
@@
 			)
 		)
-		(property "Value" "14.7k"
+		(property "Value" "15k"
 			(at 168.91 204.4699 0)
 			(effects
@@
 			)
 		)
-		(property "Value" "51k"
+		(property "Value" "56k"
 			(at 133.35 121.9199 0)
 			(effects
@@
 			)
 		)
-		(property "Value" "27.1k"
+		(property "Value" "27k"
 			(at 184.15 191.7699 0)
 			(effects
@@
 			)
 		)
-		(property "Value" "36.2k"
+		(property "Value" "39k"
 			(at 195.58 54.6099 0)
 			(effects
