File: Schematic_PCB/Music_Visualizer/Music_Visualizer.kicad_sch (KiCad schematic)
At the start: 137 parts, among them U1 LM324, U2 LM324, U3 LM324, U4 LM324, U5 LM324, U6 LM324, U7 LM324

Commit message: Remove jacks and compact placement
Parts:
- C17, C24, C43: footprint Capacitor_SMD:CP_Elec_4x5.4 -> Custom_Footprints:C_0805_2012Metric_Pad1.18x1.45mm_HandSolder
Connections:
- net VSubBass: now also C43.1; no longer C43.2
- net at C5.2, R9.1, U1.8: now also C43.2; no longer C43.1
Other:
- moved on the sheet: C43
Changed lines of the file:
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@@
 			)
 		)
-		(property "Footprint" "Capacitor_SMD:CP_Elec_4x5.4"
+		(property "Footprint" "Custom_Footprints:C_0805_2012Metric_Pad1.18x1.45mm_HandSolder"
 			(at 213.36 183.1848 0)
 			(effects
@@
 			)
 		)
-		(property "Footprint" "Capacitor_SMD:CP_Elec_4x5.4"
+		(property "Footprint" "Custom_Footprints:C_0805_2012Metric_Pad1.18x1.45mm_HandSolder"
 			(at 213.36 113.3348 0)
 			(effects
@@
 	(symbol
 		(lib_id "Device:C")
-		(at 220.98 46.99 90)
+		(at 220.98 46.99 270)
+		(mirror x)
 		(unit 1)
 		(exclude_from_sim no)
@@
 		(on_board yes)
 		(dnp no)
-		(fields_autoplaced yes)
 		(property "Reference" "C43"
 			(at 220.98 39.37 90)
@@
 			)
 		)
-		(property "Footprint" "Capacitor_SMD:CP_Elec_4x5.4"
-			(at 224.79 46.0248 0)
+		(property "Footprint" "Custom_Footprints:C_0805_2012Metric_Pad1.18x1.45mm_HandSolder"
+			(at 217.17 46.0248 0)
 			(effects
 				(font

Commit message: pre RDC
Parts:
- C1, C11, C12, C13, C14, C15, C16, C17, C18, C19, C2, C20, C21, C22, C23, C24, C25, C26, C27, C28, C29, C3, C30, C31, C32, C33, C34, C35, C36, C37, C38, C39, C4, C40, C41, C42, C43, C44, C45, C46, C47, C48, C49, C5, C50, C51, C52, C53, C6: footprint Custom_Footprints:C_0805_2012Metric_Pad1.18x1.45mm_HandSolder -> Custom_Footprints:custom_C_0805_2012Metric_Pad1.18x1.45mm_HandSolder
- H1, H2, H3, H4: footprint MountingHole:MountingHole_3.2mm_M3 -> Custom_Footprints:Apgriezts_MountingHole_2.2mm_M2
- TP1, TP2, TP3, TP4, TP5, TP6, TP7: footprint Custom_Footprints:TEST1Y -> Custom_Footprints:NEW_2_TestPoint_Loop_D2.60mm_Drill0.9mm_Beaded
