File: Schematic_PCB/Music_Visualizer/Music_Visualizer.kicad_sch (KiCad schematic)
At the start: 137 parts, among them U1 LM324, U2 LM324, U3 LM324, U4 LM324, U5 LM324, U6 LM324, U7 LM324

Commit message: Replace filters with Chebyshev
Parts:
- C39, C40, C41, C42, C44, C45: value 4.7n -> 2.2n
- C47, C48, C49, C50, C51, C52: value 2.2n -> 330p
- R1: value 27k -> 30k
- R15: value 120k -> 51k
- R16: value 12k -> 24k
- R17: value 3.3k -> 4.7k
- R18: value 56k -> 200k
- R19: value 18k -> 9.1k
- R2: value 12k -> 10k
- R20: value 15k -> 1.8k
- R21: value 39k -> 68k
- R23: value 22k -> 20k
- R24: value 6.8k -> 6.2k
- R25: value 100k -> 43k
- R26: value 8.2 -> 20k
- R27: value 2.7k -> 4.3k
- R28: value 39k -> 160k
- R29: value 15k -> 6.8k
- R3: value 150k -> 56k
- R30: value 15k -> 1.5k
- R31: value 27k -> 56k
- R35: value 82k -> 36k
- R36: value 8.2k -> 18k
- R37: value 2.2k -> 3.3k
- R38: value 33k -> 130k
- R39: value 12k -> 6.2k
- R4: value 10k -> 30k
- R40: value 10k -> 1.2k
- R41: value 27k -> 47k
- R44: value 4.7k -> 4.3k
- R45: value 68k -> 30k
- R46: value 6.8k -> 15k
- R47: value 1.8k -> 3k
- R48: value 33k -> 120k
- R49: value 10k -> 5.6k
- R5: value 4.7k -> 6.8k
- R50: value 8.2 -> 1k
- R51: value 22k -> 43k
- R53: value 15k -> 30k
- R54: value 3.3k -> 7.5k
- R56: value 6.8k -> 27k
- R57: value 1.5k -> 5.1k
- R58: value 27k -> 220k
- R6: value 47k -> 240k
- R60: value 6.8k -> 1.8k
- R61: value 22k -> 82k
- R63: value 10k -> 56k
- R64: value 5.6k -> 22k
- R65: value 39k -> 120k
- R67: value 3.3k -> 20k
- R68: value 1.6k -> 4.7k
- R69: value 15k -> 150k
- R7: value 18k -> 10k
- R70: value 5.6k -> 62k
- R71: value 22k -> 16k
- R72: value 10k -> 510k
- R8: value 39k -> 2.2.k
- R9: value 39k -> 75k
Changed lines of the file:
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@@
 			)
 		)
-		(property "Value" "4.7n"
+		(property "Value" "2.2n"
 			(at 386.08 123.19 90)
 			(show_name no)
@@
 			)
 		)
-		(property "Value" "12k"
+		(property "Value" "10k"
 			(at 74.93 64.7699 0)
 			(show_name no)
@@
 			)
 		)
-		(property "Value" "6.8k"
+		(property "Value" "6.2k"
 			(at 63.5 201.9299 0)
 			(show_name no)
@@
 			)
 		)
-		(property "Value" "2.2n"
+		(property "Value" "330p"
 			(at 434.34 196.85 90)
 			(show_name no)
@@
 			)
 		)
-		(property "Value" "8.2"
+		(property "Value" "20k"
 			(at 110.49 195.58 90)
 			(show_name no)
@@
 			)
 		)
-		(property "Value" "2.2n"
+		(property "Value" "330p"
 			(at 332.74 196.85 90)
 			(show_name no)
@@
 			)
 		)
-		(property "Value" "82k"
+		(property "Value" "36k"
 			(at 83.82 265.4299 0)
 			(show_name no)
@@
 			)
 		)
-		(property "Value" "100k"
+		(property "Value" "43k"
 			(at 81.28 191.7699 0)
 			(show_name no)
@@
 			)
 		)
-		(property "Value" "22k"
+		(property "Value" "20k"
 			(at 54.61 193.04 90)
 			(show_name no)
@@
 			)
 		)
-		(property "Value" "150k"
+		(property "Value" "56k"
 			(at 92.71 54.6099 0)
 			(show_name no)
@@
 			)
 		)
-		(property "Value" "2.2k"
+		(property "Value" "3.3k"
 			(at 123.19 278.1299 0)
 			(show_name no)
@@
 			)
 		)
-		(property "Value" "3.3k"
+		(property "Value" "7.5k"
 			(at 325.12 133.3499 0)
 			(show_name no)
@@
 			)
 		)
-		(property "Value" "4.7k"
+		(property "Value" "4.3k"
 			(at 326.39 58.4199 0)
 			(show_name no)
@@
 			)
 		)
-		(property "Value" "2.2n"
+		(property "Value" "330p"
 			(at 386.08 184.15 90)
 			(show_name no)
@@
 			)
 		)
-		(property "Value" "1.5k"
+		(property "Value" "5.1k"
 			(at 382.27 135.8899 0)
 			(show_name no)
@@
 			)
 		)
-		(property "Value" "4.7n"
+		(property "Value" "2.2n"
 			(at 332.74 123.19 90)
 			(show_name no)
@@
 			)
 		)
-		(property "Value" "6.8k"
+		(property "Value" "27k"
 			(at 372.11 127 90)
 			(show_name no)
@@
 			)
 		)
-		(property "Value" "120k"
+		(property "Value" "51k"
 			(at 81.28 121.9199 0)
 			(show_name no)
@@
 			)
 		)
-		(property "Value" "15k"
+		(property "Value" "1.8k"
 			(at 168.91 134.6199 0)
 			(show_name no)
@@
 			)
 		)
-		(property "Value" "6.8k"
+		(property "Value" "1.8k"
 			(at 430.53 135.8899 0)
 			(show_name no)
@@
 			)
 		)
-		(property "Value" "2.7k"
+		(property "Value" "4.3k"
 			(at 120.65 204.4699 0)
 			(show_name no)
@@
 			)
 		)
-		(property "Value" "18k"
+		(property "Value" "10k"
 			(at 170.18 58.42 90)
 			(show_name no)
@@
 			)
 		)
-		(property "Value" "22k"
+		(property "Value" "16k"
 			(at 430.53 209.5499 0)
 			(show_name no)
@@
 			)
 		)
-		(property "Value" "3.3k"
+		(property "Value" "4.7k"
 			(at 120.65 134.6199 0)
 			(show_name no)
@@
 			)
 		)
-		(property "Value" "6.8k"
+		(property "Value" "15k"
 			(at 373.38 52.07 90)
 			(show_name no)
@@
 			)
 		)
-		(property "Value" "33k"
+		(property "Value" "130k"
 			(at 135.89 265.4299 0)
 			(show_name no)
@@
 			)
 		)
-		(property "Value" "10k"
+		(property "Value" "30k"
 			(at 121.92 58.42 90)
 			(show_name no)
@@
 			)
 		)
-		(property "Value" "22k"
+		(property "Value" "82k"
 			(at 445.77 123.1899 0)
 			(show_name no)
@@
 			)
 		)
-		(property "Value" "12k"
+		(property "Value" "24k"
 			(at 110.49 125.73 90)
 			(show_name no)
@@
 			)
 		)
-		(property "Value" "27k"
+		(property "Value" "47k"
 			(at 186.69 265.4299 0)
 			(show_name no)
@@
 			)
 		)
-		(property "Value" "27k"
+		(property "Value" "220k"
 			(at 394.97 123.1899 0)
 			(show_name no)
@@
 			)
 		)
-		(property "Value" "3.3k"
+		(property "Value" "20k"
 			(at 372.11 200.66 90)
 			(show_name no)
@@
 			)
 		)
-		(property "Value" "5.6k"
+		(property "Value" "22k"
 			(at 325.12 207.0099 0)
 			(show_name no)
@@
 			)
 		)
-		(property "Value" "1.6k"
+		(property "Value" "4.7k"
 			(at 382.27 209.5499 0)
 			(show_name no)
@@
 			)
 		)
-		(property "Value" "4.7k"
+		(property "Value" "6.8k"
 			(at 132.08 67.3099 0)
 			(show_name no)
@@
 			)
 		)
-		(property "Value" "33k"
+		(property "Value" "120k"
 			(at 396.24 48.2599 0)
 			(show_name no)
@@
 			)
 		)
-		(property "Value" "4.7n"
+		(property "Value" "2.2n"
 			(at 434.34 123.19 90)
 			(show_name no)
@@
 			)
 		)
-		(property "Value" "8.2"
+		(property "Value" "1k"
 			(at 431.8 60.9599 0)
 			(show_name no)
@@
 			)
 		)
-		(property "Value" "15k"
+		(property "Value" "150k"
 			(at 394.97 196.8499 0)
 			(show_name no)
@@
 			)
 		)
-		(property "Value" "39k"
+		(property "Value" "160k"
 			(at 133.35 191.7699 0)
 			(show_name no)
@@
 			)
 		)
-		(property "Value" "1.8k"
+		(property "Value" "3k"
 			(at 383.54 60.9599 0)
 			(show_name no)
@@
 			)
 		)
-		(property "Value" "10k"
+		(property "Value" "1.2k"
 			(at 171.45 278.1299 0)
 			(show_name no)
@@
 			)
 		)
-		(property "Value" "68k"
+		(property "Value" "30k"
 			(at 344.17 48.2599 0)
 			(show_name no)
@@
 			)
 		)
-		(property "Value" "5.6k"
+		(property "Value" "62k"
 			(at 420.37 200.66 90)
 			(show_name no)
@@
 			)
 		)
-		(property "Value" "12k"
+		(property "Value" "6.2k"
 			(at 161.29 269.24 90)
 			(show_name no)
@@
 			)
 		)
-		(property "Value" "10k"
+		(property "Value" "5.6k"
 			(at 421.64 52.07 90)
 			(show_name no)
@@
 			)
 		)
-		(property "Value" "39k"
+		(property "Value" "68k"
 			(at 184.15 121.9199 0)
 			(show_name no)
@@
 			)
 		)
-		(property "Value" "39k"
+		(property "Value" "120k"
 			(at 342.9 196.8499 0)
 			(show_name no)
@@
 			)
 		)
-		(property "Value" "18k"
+		(property "Value" "9.1k"
 			(at 158.75 125.73 90)
 			(show_name no)
@@
 			)
 		)
-		(property "Value" "10k"
+		(property "Value" "56k"
 			(at 316.23 198.12 90)
 			(show_name no)
@@
 			)
 		)
-		(property "Value" "15k"
+		(property "Value" "6.8k"
 			(at 158.75 195.58 90)
 			(show_name no)
@@
 			)
 		)
-		(property "Value" "2.2n"
+		(property "Value" "330p"
 			(at 332.74 184.15 90)
 			(show_name no)
@@
 			)
 		)
-		(property "Value" "27k"
+		(property "Value" "30k"
 			(at 66.04 55.88 90)
 			(show_name no)
@@
 			)
 		)
-		(property "Value" "22k"
+		(property "Value" "43k"
 			(at 447.04 48.2599 0)
 			(show_name no)
@@
 			)
 		)
-		(property "Value" "15k"
+		(property "Value" "30k"
 			(at 316.23 124.46 90)
 			(show_name no)
@@
 			)
 		)
-		(property "Value" "39k"
+		(property "Value" "2.2.k"
 			(at 180.34 67.3099 0)
 			(show_name no)
@@
 			)
 		)
-		(property "Value" "8.2k"
+		(property "Value" "18k"
 			(at 113.03 269.24 90)
 			(show_name no)
@@
 			)
 		)
-		(property "Value" "10k"
+		(property "Value" "510k"
 			(at 445.77 196.8499 0)
 			(show_name no)
@@
 			)
 		)
-		(property "Value" "47k"
+		(property "Value" "240k"
 			(at 144.78 54.6099 0)
 			(show_name no)
@@
 			)
 		)
-		(property "Value" "2.2n"
+		(property "Value" "330p"
 			(at 386.08 196.85 90)
 			(show_name no)
@@
 			)
 		)
-		(property "Value" "4.7n"
+		(property "Value" "2.2n"
 			(at 434.34 110.49 90)
 			(show_name no)
@@
 			)
 		)
-		(property "Value" "15k"
+		(property "Value" "1.5k"
 			(at 168.91 204.4699 0)
 			(show_name no)
@@
 			)
 		)
-		(property "Value" "4.7n"
+		(property "Value" "2.2n"
 			(at 386.08 110.49 90)
 			(show_name no)
@@
 			)
 		)
-		(property "Value" "4.7n"
+		(property "Value" "2.2n"
 			(at 332.74 110.49 90)
 			(show_name no)
@@
 			)
 		)
-		(property "Value" "56k"
+		(property "Value" "200k"
 			(at 133.35 121.9199 0)
 			(show_name no)
@@
 			)
 		)
-		(property "Value" "27k"
+		(property "Value" "56k"
 			(at 184.15 191.7699 0)
 			(show_name no)
@@
 			)
 		)
-		(property "Value" "39k"
+		(property "Value" "75k"
 			(at 195.58 54.6099 0)
 			(show_name no)
@@
 			)
 		)
-		(property "Value" "2.2n"
+		(property "Value" "330p"
 			(at 434.34 184.15 90)
 			(show_name no)
