File: Schematic_PCB/Music_Visualizer/Power.kicad_sch (KiCad schematic)
At the start: 38 parts, among them J6 3.5mm, J7 Barrel_Jack_PTH_Slot, Q1 DMP2123LQ-7, SW2 SW_SPST, U1 LM324, U2 LM324, U3 LM324, U4 LM324, U5 LM324, U6 LM324, U7 LM324, U8 LM324

Commit message: Battery low
Parts:
- removed J7: Barrel_Jack_PTH_Slot, PCM_SparkFun-Connector:Barrel_Jack_PTH_Slot, symbol PCM_SparkFun-Connector:Barrel_Jack_PTH_Slot
- added J2: Barrel_Jack_PTH, Custom_Footprints:RAPC722X, symbol PCM_SparkFun-Connector:Barrel_Jack_PTH
Connections:
- net GND: now also J2.1 (PWR)
- net at Q1.1 (D): now also J2.2 (GND)
- net at J6.1 (Pin_1), TP10.1: now also J2.3 (GNDBREAK)
Changed lines of the file:
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@@
 	(wire
 		(pts
-			(xy 160.02 54.61) (xy 166.37 54.61)
+			(xy 152.4 54.61) (xy 166.37 54.61)
 		)
 		(stroke
@@
 	(wire
 		(pts
-			(xy 160.02 52.07) (xy 181.61 52.07)
+			(xy 152.4 52.07) (xy 181.61 52.07)
 		)
 		(stroke
@@
 	(wire
 		(pts
-			(xy 160.02 57.15) (xy 161.29 57.15)
+			(xy 152.4 57.15) (xy 161.29 57.15)
 		)
 		(stroke
@@
 	)
 	(symbol
+		(lib_id "PCM_SparkFun-Connector:Barrel_Jack_PTH")
+		(at 144.78 54.61 0)
+		(mirror x)
+		(unit 1)
+		(exclude_from_sim no)
+		(in_bom yes)
+		(on_board yes)
+		(dnp no)
+		(property "Reference" "J2"
+			(at 144.78 63.5 0)
+			(effects
+				(font
+					(size 1.27 1.27)
+				)
+			)
+		)
+		(property "Value" "Barrel_Jack_PTH"
+			(at 144.78 60.96 0)
+			(effects
+				(font
+					(size 1.27 1.27)
+				)
+			)
+		)
+		(property "Footprint" "Custom_Footprints:RAPC722X"
+			(at 146.05 45.72 0)
+			(effects
+				(font
+					(size 1.27 1.27)
+				)
+				(hide yes)
+			)
+		)
+		(property "Datasheet" "https://www.sparkfun.com/datasheets/Prototyping/Barrel-Connector-PJ-202A.pdf"
+			(at 146.05 43.18 0)
+			(effects
+				(font
+					(size 1.27 1.27)
+				)
+				(hide yes)
+			)
+		)
+		(property "Description" "DC Barrel Jack with an internal switch"
+			(at 144.78 40.64 0)
+			(effects
+				(font
+					(size 1.27 1.27)
+				)
+				(hide yes)
+			)
+		)
+		(property "PROD_ID" "CONN-08197"
+			(at 144.78 46.99 0)
+			(effects
+				(font
+					(size 1.27 1.27)
+				)
+				(hide yes)
+			)
+		)
+		(pin "1"
+		)
+		(pin "3"
+		)
+		(pin "2"
+		)
+		(instances
+			(project ""
+				(path "/236ff8a0-79ed-4eaf-ae36-90444797fa8d/d77592bc-5812-4255-9ac4-28fcc93efec5"
+					(reference "J2")
+					(unit 1)
+				)
+			)
+		)
+	)
+	(symbol
 		(lib_id "Device:C_Polarized")
 		(at 220.98 55.88 0)
@@
 					(unit 1)
 				)
-			)
-		)
-	)
-	(symbol
-		(lib_id "PCM_SparkFun-Connector:Barrel_Jack_PTH_Slot")
-		(at 152.4 54.61 0)
-		(mirror x)
-		(unit 1)
-		(exclude_from_sim no)
-		(in_bom yes)
-		(on_board yes)
-		(dnp no)
-		(property "Reference" "J7"
-			(at 152.4 63.5 0)
-			(effects
-				(font
-					(size 1.27 1.27)
-				)
-			)
-		)
-		(property "Value" "Barrel_Jack_PTH_Slot"
-			(at 152.4 60.96 0)
-			(effects
-				(font
-					(size 1.27 1.27)
-				)
-			)
-		)
-		(property "Footprint" "PCM_SparkFun-Connector:Barrel_Jack_PTH_Slot"
-			(at 152.4 44.45 0)
-			(effects
-				(font
-					(size 1.27 1.27)
-				)
-				(hide yes)
-			)
-		)
-		(property "Datasheet" "https://www.sparkfun.com/datasheets/Prototyping/Barrel-Connector-PJ-202A.pdf"
-			(at 152.4 41.91 0)
-			(effects
-				(font
-					(size 1.27 1.27)
-				)
-				(hide yes)
-			)
-		)
-		(property "Description" "DC Barrel Jack with an internal switch"
-			(at 152.4 39.37 0)
-			(effects
-				(font
-					(size 1.27 1.27)
-				)
-				(hide yes)
-			)
-		)
-		(property "PROD_ID" "CONN-08197"
-			(at 152.4 46.99 0)
-			(effects
-				(font
-					(size 1.27 1.27)
-				)
-				(hide yes)
-			)
-		)
-		(pin "PWR"
-		)
-		(pin "GNDBREAK"
-		)
-		(pin "GND"
-		)
-		(instances
-			(project ""
-				(path "/236ff8a0-79ed-4eaf-ae36-90444797fa8d/d77592bc-5812-4255-9ac4-28fcc93efec5"
-					(reference "J7")
-					(unit 1)
-				)

Commit message: PCB V1 done
Parts:
- C55, C59, C60, C61, C62, C63, C64, C65, C66, C67, C68, C69, C70, C71, C72, C73, C74: footprint Capacitor_SMD:C_0805_2012Metric_Pad1.18x1.45mm_HandSolder -> Custom_Footprints:C_0805_2012Metric_Pad1.18x1.45mm_HandSolder
- R82, R83, R84: footprint Resistor_SMD:R_0805_2012Metric_Pad1.20x1.40mm_HandSolder -> Custom_Footprints:R_0805_2012Metric_Pad1.20x1.40mm_HandSolder
