File: Schematic_PCB/Music_Visualizer/audio_signal.kicad_sch (KiCad schematic)
At the start: 17 parts, among them J1 NMJ4HCD2, J3 Screw_Terminal_01x02, J4 NMJ4HCD2, J5 Screw_Terminal_01x02, SW1 SW_Slide_DPDT, U8 LM324

Commit message: pre RDC
Parts:
- C10, C8: footprint Capacitor_THT:CP_Radial_D5.0mm_P2.00mm -> Capacitor_SMD:CP_Elec_4x5.4
- C7, C9: footprint Custom_Footprints:C_0805_2012Metric_Pad1.18x1.45mm_HandSolder -> Custom_Footprints:custom_C_0805_2012Metric_Pad1.18x1.45mm_HandSolder
- J3, J5: footprint TerminalBlock_Phoenix:TerminalBlock_Phoenix_MPT-0,5-2-2.54_1x02_P2.54mm_Horizontal -> Connector_JST:JST_EH_B2B-EH-A_1x02_P2.50mm_Vertical
- T_in1: renamed from TP8; value T_a_in -> T_in; footprint Custom_Footprints:TEST1Y -> Custom_Footprints:NEW_2_TestPoint_Loop_D2.60mm_Drill0.9mm_Beaded
- T_out1: renamed from TP14; value T_a_out -> T_out; footprint Custom_Footprints:TEST1Y -> Custom_Footprints:NEW_2_TestPoint_Loop_D2.60mm_Drill0.9mm_Beaded
- T_sig1: renamed from TP9; footprint Custom_Footprints:TEST1Y -> Custom_Footprints:NEW_2_TestPoint_Loop_D2.60mm_Drill0.9mm_Beaded
Changed lines of the file:
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@@
 			)
 		)
-		(property "Footprint" "Custom_Footprints:C_0805_2012Metric_Pad1.18x1.45mm_HandSolder"
+		(property "Footprint" "Custom_Footprints:custom_C_0805_2012Metric_Pad1.18x1.45mm_HandSolder"
 			(at 100.33 124.7648 0)
 			(hide yes)
@@
 			)
 		)
-		(property "Footprint" "Capacitor_THT:CP_Radial_D5.0mm_P2.00mm"
+		(property "Footprint" "Capacitor_SMD:CP_Elec_4x5.4"
 			(at 142.24 127.3048 0)
 			(hide yes)
@@
 		(in_pos_files yes)
 		(dnp no)
-		(property "Reference" "TP14"
+		(property "Reference" "T_out1"
 			(at 158.75 135.89 0)
 			(show_name no)
@@
 			)
 		)
-		(property "Value" "T_a_out"
+		(property "Value" "T_out"
 			(at 158.75 133.35 0)
 			(show_name no)
@@
 			)
 		)
-		(property "Footprint" "Custom_Footprints:TEST1Y"
+		(property "Footprint" "Custom_Footprints:NEW_2_TestPoint_Loop_D2.60mm_Drill0.9mm_Beaded"
 			(at 165.1 223.19 0)
 			(hide yes)
@@
 			(project "Music_Visualizer"
 				(path "/236ff8a0-79ed-4eaf-ae36-90444797fa8d/c910a8c7-0bf8-4b44-820c-85a625c5ccef"
-					(reference "TP14")
+					(reference "T_out1")
 					(unit 1)
 				)
@@
 			)
 		)
-		(property "Footprint" "TerminalBlock_Phoenix:TerminalBlock_Phoenix_MPT-0,5-2-2.54_1x02_P2.54mm_Horizontal"
+		(property "Footprint" "Connector_JST:JST_EH_B2B-EH-A_1x02_P2.50mm_Vertical"
 			(at 201.93 52.07 0)
 			(hide yes)
@@
 			)
 		)
-		(property "Footprint" "Capacitor_THT:CP_Radial_D5.0mm_P2.00mm"
+		(property "Footprint" "Capacitor_SMD:CP_Elec_4x5.4"
 			(at 135.89 46.0248 0)
 			(hide yes)
@@
 			)
 		)
-		(property "Footprint" "Custom_Footprints:C_0805_2012Metric_Pad1.18x1.45mm_HandSolder"
+		(property "Footprint" "Custom_Footprints:custom_C_0805_2012Metric_Pad1.18x1.45mm_HandSolder"
 			(at 105.41 43.4848 0)
 			(hide yes)
@@
 			)
 		)
-		(property "Footprint" "TerminalBlock_Phoenix:TerminalBlock_Phoenix_MPT-0,5-2-2.54_1x02_P2.54mm_Horizontal"
+		(property "Footprint" "Connector_JST:JST_EH_B2B-EH-A_1x02_P2.50mm_Vertical"
 			(at 54.61 52.07 0)
 			(hide yes)
@@
 		(dnp no)
 		(fields_autoplaced yes)
-		(property "Reference" "TP8"
+		(property "Reference" "T_in1"
 			(at 86.36 36.83 0)
 			(show_name no)
@@
 			)
 		)
-		(property "Value" "T_a_in"
+		(property "Value" "T_in"
 			(at 86.36 39.37 0)
 			(show_name no)
@@
 			)
 		)
-		(property "Footprint" "Custom_Footprints:TEST1Y"
+		(property "Footprint" "Custom_Footprints:NEW_2_TestPoint_Loop_D2.60mm_Drill0.9mm_Beaded"
 			(at 80.01 139.37 0)
 			(hide yes)
@@
 			(project "Music_Visualizer"
 				(path "/236ff8a0-79ed-4eaf-ae36-90444797fa8d/c910a8c7-0bf8-4b44-820c-85a625c5ccef"
-					(reference "TP8")
+					(reference "T_in1")
 					(unit 1)
 				)
@@
 		(dnp no)
 		(fields_autoplaced yes)
-		(property "Reference" "TP9"
+		(property "Reference" "T_sig1"
 			(at 40.64 83.82 0)
 			(show_name no)
@@
 			)
 		)
-		(property "Footprint" "Custom_Footprints:TEST1Y"
+		(property "Footprint" "Custom_Footprints:NEW_2_TestPoint_Loop_D2.60mm_Drill0.9mm_Beaded"
 			(at 34.29 186.36 0)
 			(hide yes)
@@
 			(project "Music_Visualizer"
 				(path "/236ff8a0-79ed-4eaf-ae36-90444797fa8d/c910a8c7-0bf8-4b44-820c-85a625c5ccef"
-					(reference "TP9")
+					(reference "T_sig1")
 					(unit 1)
 				)
